Commit message: mechatronics system and IMU

File: urdf/AMR_model.urdf (robot description, URDF)
Before this commit: robot AGV, 5 links, 4 joints
Links:
- removed link IMU
- added link imu_link; visual box size=0.5 0.2 0.1
Joints:
- joint imu_joint: child IMU -> imu_link

Commit message: add(AMR_model.urdf, mechatronics.launch):add velodyne launch, change urdf velodyne frame id

File: urdf/AMR_model.urdf (robot description, URDF)
Before this commit: robot AGV, 5 links, 4 joints
Links:
- removed link VLP16
- added link VLP16_link; visual mesh filename=package://scl_amr/meshes/sick_tim_5xx.stl scale=0.01 0.01 0.01
Joints:
- joint VLP16_joint: child VLP16 -> VLP16_link

Commit message: fast_lio

File: urdf/AMR_model.urdf (robot description, URDF)
Before this commit: robot AGV, 5 links, 4 joints
Links:
- removed link VLP16_link
- added link velodyne; visual mesh filename=package://scl_amr/meshes/sick_tim_5xx.stl scale=0.01 0.01 0.01
Joints:
- removed joint VLP16_joint
- added joint velodyne: type fixed, parent base_link, child velodyne, origin xyz=0.35 0 1.26 rpy=0 0 0
